File: kicad/sawtooth.kicad_pcb (KiCad board)
At the start: 4 copper layers, 63.3 x 31.8 mm, 29 parts, among them J1 Conn_02x04_Odd_Even, J2 Conn_Coaxial, J3 Conn_Coaxial, J4 Conn_01x05_Pin, J6 Conn_01x06_Pin, J7 AVR-TPI-6, U1 DS1020, U2 TLV1117-33, U4 74LVC125, U5 ATtiny102-SS

Commit message: board layout done
Parts:
- removed R2, R9: 0, Resistor_SMD:R_0805_2012Metric_Pad1.20x1.40mm_HandSolder
- added C6: 1u, Capacitor_SMD:C_0805_2012Metric_Pad1.18x1.45mm_HandSolder, F.Cu at (152.8, 114.2)
- added C7: 1u, Capacitor_SMD:C_0805_2012Metric_Pad1.18x1.45mm_HandSolder, F.Cu at (150.9, 102.9)
- H1, H2, H3, H4: footprint MountingHole:MountingHole_3.2mm_M3_DIN965_Pad_TopBottom -> MountingHole:MountingHole_3mm_Pad_TopBottom
- J1: moved to B.Cu
- moved J6 71.6 mm to (150.5, 117.0), turned to 90 degrees
- moved D1 64.8 mm to (123.9, 114.4)
- moved J3 64.8 mm to (163.7, 92.2)
- moved U2 61.6 mm to (117.2, 101.7), turned to 180 degrees
- moved U1 58.5 mm to (142.5, 107.1)
- moved R4 53.6 mm to (124.9, 106.6), turned to 90 degrees
- moved R3 50.1 mm to (133.9, 102.5), turned to 90 degrees
- moved R1 47.3 mm to (135.3, 94.0), turned to 90 degrees
- moved C1 46.3 mm to (128.1, 106.6), turned to -90 degrees
- moved C4 45.1 mm to (117.0, 106.7)
- moved R6 43.2 mm to (163.7, 100.2), turned to -90 degrees
- moved C3 43.2 mm to (157.2, 113.0)
- moved J7 42.9 mm to (126.0, 90.0), turned to -90 degrees
- moved R5 42.6 mm to (155.8, 99.9), turned to -90 degrees
- moved R7 41.4 mm to (150.6, 105.8), turned to 180 degrees
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Connections:
- net Net-(J2-In) renamed /PPS_COMP_OUT
- net Net-(J3-In) renamed /PPS_RAW_OUT
- net Net-(R5-Pad2) renamed /PPS_DELAY_OUT_BUF
- net Net-(U1-OUT) renamed /PPS_DELAY_OUT
- J4 pad 2: TO_GPS_DATA -> FROM_GPS_DATA
- J4 pad 3: FROM_GPS_DATA -> TO_GPS_DATA
- U1 pad 1: Net-(U1-IN) -> /PPS_DELAY_IN
- U2 pad 4: (no net) -> +3.3V
- U4 pad 11: PPS_RAW -> /PPS_DELAY_IN
- U4 pad 12: Net-(U4-Pad12) -> /PPS_IN
- U4 pad 3: Net-(U1-IN) -> /RAW_BUF
- U4 pad 5: /PPS_IN -> /RAW_BUF
- U4 pad 6: Net-(U4-Pad12) -> PPS_RAW
Routing:
- net TO_GPS_DATA: track 0.00 -> 67.9 mm, vias 0 -> 1
- net FROM_GPS_DATA: track 0.00 -> 65.1 mm, vias 0 -> 1
- net MOSI: track 0.00 -> 44.2 mm
- net SCK: track 0.00 -> 37.8 mm
- net SS: track 0.00 -> 31.5 mm
- net /PPS_IN: track 0.00 -> 25.5 mm
- net /LED: track 0.00 -> 25.4 mm, vias 0 -> 2
- net /AT_TXD: track 0.00 -> 23.7 mm
- net GND: track 0.00 -> 22.9 mm, vias 0 -> 19
- net /PPS_DELAY_IN: track 0.00 -> 19.8 mm
- net +3.3V: track 0.00 -> 17.8 mm, vias 0 -> 13
- net /AT_RXD: track 0.00 -> 10.1 mm
- net /PPS_DELAY_OUT: track 0.00 -> 8.15 mm
- net /LED_R: track 0.00 -> 7.00 mm
- net /PPS_COMP_OUT: track 0.00 -> 6.89 mm
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- added copper zone on F.Cu, net +3.3V
- added copper zone on In2.Cu, net +3.3V
- added copper zone on F.Cu, net GND
- added copper zone on In1.Cu, net GND
- added copper zone on F.Cu, net VBUS
- added copper zone on In2.Cu, net VBUS
Other:
- board size 63.3 x 31.8 mm -> 66.1 x 31.8 mm
