File: kicad/sawtooth.kicad_sch (KiCad schematic)
At the start: 23 parts, among them J1 Conn_02x04_Odd_Even, J2 Conn_Coaxial, J3 Conn_Coaxial, J4 Conn_01x04_Pin, J5 AVR-ISP-6, J6 Conn_01x06_Pin, U1 DS1020, U2 TLV1117-33, U3 ATtiny85-20S, U4 74LVC125

Commit message: update and board start
Parts:
- removed J4: Conn_01x04_Pin, Connector_PinHeader_2.54mm:PinHeader_1x04_P2.54mm_Vertical, symbol Connector:Conn_01x04_Pin
- removed J5: AVR-ISP-6, Connector_PinHeader_2.54mm:PinHeader_2x03_P2.54mm_Vertical, symbol Connector:AVR-ISP-6
- removed U3: ATtiny85-20S, Package_SO:SOIC-8W_5.3x5.3mm_P1.27mm, symbol MCU_Microchip_ATtiny:ATtiny85-20S
- added H1, H2, H3, H4: MountingHole_Pad, MountingHole:MountingHole_3.2mm_M3_DIN965_Pad_TopBottom, symbol Mechanical:MountingHole_Pad
- added J4: Conn_01x05_Pin, Connector_PinHeader_2.54mm:PinHeader_1x05_P2.54mm_Vertical, symbol Connector:Conn_01x05_Pin
- added J7: AVR-TPI-6, Connector_PinHeader_2.54mm:PinHeader_2x03_P2.54mm_Vertical, symbol Connector:AVR-TPI-6
- added R8, R9: 0, Resistor_SMD:R_0805_2012Metric_Pad1.20x1.40mm_HandSolder, symbol Device:R_US
- added U5: ATtiny102-SS, Package_SO:SOIC-8_3.9x4.9mm_P1.27mm, symbol MCU_Microchip_ATtiny:ATtiny102-SS
- J2, J3: footprint (none) -> Connector_Coaxial:SMA_Amphenol_901-143_Horizontal
Connections:
- net ISP_RSTL is gone; now on net SS: R3.1
- net +3.3V: now also U5.1 (VCC)
- net FROM_GPS_DATA: now also R1.2, J4.3 (Pin_3), R9.1; no longer R1.1
- net GND: now also H1.1, H2.1, H3.1, H4.1, J4.5 (Pin_5), J7.6 (GND), U5.8 (GND); no longer U4.12
- net PPS_RAW: now also U4.11; no longer U4.6
- net SS: now also J7.5 (~{RST}), U5.4 (~{RESET}/PA2)
- net TO_GPS_DATA: now also J4.2 (Pin_2), R8.2
- net VBUS: now also J4.1 (Pin_1), J7.2 (VCC)
- net LED_R: now reaches D1.2 (A), R4.1
- net LED: now reaches D1.1 (K)
- net LED: now also U5.5 (PB1)
- net ISP_MISO renamed MOSI
- net MOSI: now also J7.1 (DATA), U5.3 (PA1)
- net ISP_MOSI renamed AT_RXD
- net AT_RXD: now also R1.1, U5.7 (PB3); no longer R1.2
- net ISP_SCK renamed SCK
- net SCK: now also J7.3 (CLOCK), U5.2 (PA0)
- new net: U4.12, U4.6
- new net AT_TXD: J4.4 (Pin_4), R8.1, R9.2, U5.6 (PB2)
- no-connect marks 11 -> 10
Other:
- moved on the sheet: C1, C2, C3, C4, C5, D1, J1, J2, J3, J6, R1, R2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

Commit message: board layout done
Parts:
- removed R2, R9: 0, Resistor_SMD:R_0805_2012Metric_Pad1.20x1.40mm_HandSolder, symbol Device:R_US
- added C6, C7: 1u, Capacitor_SMD:C_0805_2012Metric_Pad1.18x1.45mm_HandSolder, symbol Device:C
- H1, H2, H3, H4: footprint MountingHole:MountingHole_3.2mm_M3_DIN965_Pad_TopBottom -> MountingHole:MountingHole_3mm_Pad_TopBottom
Connections:
- net +3.3V: now also U2.4 (VO), C6.1, C7.1
- net FROM_GPS_DATA: now also J4.2 (Pin_2); no longer J4.3 (Pin_3)
- net GND: now also C6.2, C7.2
- net PPS_IN: now also U4.12; no longer U4.5
- net PPS_RAW: now also U4.6; no longer U4.11
- net TO_GPS_DATA: now also J4.3 (Pin_3); no longer J4.2 (Pin_2)
- net PPS_RAW_OUT: now reaches J3.1 (In), R6.1
- net PPS_COMP_OUT: now reaches J2.1 (In), R5.1
- net PPS_DELAY_OUT_BUF: now reaches R5.2, U4.8
- net PPS_DELAY_IN: now reaches U1.1 (IN)
- net PPS_DELAY_IN: now also U4.11; no longer U4.3
- net PPS_DELAY_OUT: now reaches U1.15 (OUT), U4.9
- new net RAW_BUF: U4.3, U4.5
Other:
- moved on the sheet: J2, J3, U4A, U4C, U4D
